Commit message: ROS2 Jazzy and Gazebo Harmonic migration work

File: nps_uw_multibeam_sonar/urdf/multibeam_sonar_blueview_p900.xacro (robot description, xacro)
@@ -7,5 +7,5 @@
         <mass value="4.35"/>
         <pose xyz="0 0 0" rpy="0 0 0"/>
-        <inertia ixx="0.0360" ixy="0" ixz="0" iyy="0" iyz="0" izz="0.0360"/>
+        <inertia ixx="0.0360" ixy="0" ixz="0" iyy="0.0360" iyz="0" izz="0.0360"/>
       </inertial>
       <visual>
@@ -17,5 +17,5 @@
       <collision>
         <geometry>
-          <mesh filename="model://blueview_p900_nps_multibeam/meshes/COLLISION-p900.dae" scale="${scale}"/>
+          <box size="0.35 0.16 0.12"/>
         </geometry>
         <pose xyz="0 0 0" rpy="0 0 0"/>
@@ -54,5 +54,5 @@
           </save> -->
         </camera>
-        <plugin filename="libnps_multibeam_sonar_ros_plugin.so" name="${name}_sensor_controller">
+        <plugin filename="libnps_multibeam_sonar_ros_plugin.so" name="nps_uw_multibeam_sonar::NpsGazeboRosMultibeamSonar">
           <!-- Sonar properties -->
           <verticalFOV>90</verticalFOV>
@@ -131,5 +131,5 @@
           </noise>
         </ray>
-        <plugin filename="libnps_multibeam_sonar_ray_ros_plugin.so" name="${name}_sensor_controller">
+        <plugin filename="libnps_multibeam_sonar_ray_ros_plugin.so" name="nps_uw_multibeam_sonar::NpsGazeboRosMultibeamSonarRay">
           <!-- Sonar properties -->
           <verticalFOV>90</verticalFOV>

File: rexrov2/rexrov2_description/robots/rexrov2_default.xacro (robot description, xacro)
@@ -30,5 +30,5 @@
     -->
     <gazebo>
-      <plugin name="uuv_plugin" filename="libuuv_underwater_object_ros_plugin.so">
+      <plugin name="uuv_simulator_ros::UnderwaterObjectROSPlugin" filename="libuuv_underwater_object_ros_plugin.so">
         <fluid_density>1028.0</fluid_density>
         <flow_velocity_topic>hydrodynamics/current_velocity</flow_velocity_topic>

File: rexrov2/rexrov2_description/robots/rexrov2_oberon4.xacro (robot description, xacro)
@@ -29,5 +29,5 @@
      allow the addition of external models of manipulator units -->
     <gazebo>
-      <plugin name="uuv_plugin" filename="libuuv_underwater_object_ros_plugin.so">
+      <plugin name="uuv_simulator_ros::UnderwaterObjectROSPlugin" filename="libuuv_underwater_object_ros_plugin.so">
         <fluid_density>1028.0</fluid_density>
         <flow_velocity_topic>hydrodynamics/current_velocity</flow_velocity_topic>

File: rexrov2/rexrov2_description/robots/rexrov2_oberon7.xacro (robot description, xacro)
@@ -29,5 +29,5 @@
      allow the addition of external models of manipulator units -->
     <gazebo>
-      <plugin name="uuv_plugin" filename="libuuv_underwater_object_ros_plugin.so">
+      <plugin name="uuv_simulator_ros::UnderwaterObjectROSPlugin" filename="libuuv_underwater_object_ros_plugin.so">
         <fluid_density>1028.0</fluid_density>
         <flow_velocity_topic>hydrodynamics/current_velocity</flow_velocity_topic>

File: rexrov2/rexrov2_description/robots/rexrov2_oberon_arms.xacro (robot description, xacro)
@@ -30,5 +30,5 @@
      allow the addition of external models of manipulator units -->
     <gazebo>
-      <plugin name="uuv_plugin" filename="libuuv_underwater_object_ros_plugin.so">
+      <plugin name="uuv_simulator_ros::UnderwaterObjectROSPlugin" filename="libuuv_underwater_object_ros_plugin.so">
         <fluid_density>1028.0</fluid_density>
         <flow_velocity_topic>hydrodynamics/current_velocity</flow_velocity_topic>

File: rexrov2/rexrov2_description/urdf/rexrov2_sensors.xacro (robot description, xacro)
@@ -71,5 +71,14 @@
   </xacro:default_chemical_concentration_sensor_macro>
   <link name="${namespace}/sonar_link">
-    <!-- Add visual or collision elements if needed -->
+    <inertial>
+      <mass value="0.1"/>
+      <origin xyz="0 0 0" rpy="0 0 0"/>
+      <inertia ixx="0.001" ixy="0" ixz="0" iyy="0.001" iyz="0" izz="0.001"/>
+    </inertial>
+    <collision>
+      <geometry>
+        <box size="0.05 0.05 0.05"/>
+      </geometry>
+    </collision>
   </link>
    <!-- Define the Revolute Joint -->

File: uuv_simulator/uuv_gazebo_plugins/uuv_gazebo_ros_plugins/urdf/misc.xacro (robot description, xacro)
@@ -11,5 +11,5 @@
   <xacro:macro name="default_joint_state_publisher" params="namespace update_rate">
     <gazebo>
-      <plugin name="uuv_joint_state_publisher" filename="libuuv_joint_state_publisher.so">
+      <plugin name="uuv_simulator_ros::JointStatePublisher" filename="libuuv_joint_state_publisher.so">
         <robotNamespace>${namespace}</robotNamespace>
         <updateRate>${update_rate}</updateRate>

File: uuv_simulator/uuv_gazebo_plugins/uuv_gazebo_ros_plugins/urdf/thruster_snippets.xacro (robot description, xacro)
@@ -83,5 +83,5 @@
     </joint>
     <link name="${namespace}/thruster_${thruster_id}">
-      <xacro:box_inertial x="0" y="0" z="0" mass="0.001">
+      <xacro:box_inertial x="0.01" y="0.01" z="0.01" mass="0.001">
         <origin xyz="0 0 0" rpy="0 0 0"/>
       </xacro:box_inertial>
@@ -96,5 +96,5 @@
            the joint that leads to this link (and assume it to be the identity) -->
         <geometry>
-          <cylinder length="0.000001" radius="0.000001"/>
+          <cylinder length="0.01" radius="0.01"/>
         </geometry>
         <origin xyz="0 0 0" rpy="0 0 0"/>
@@ -102,5 +102,5 @@
     </link>
     <gazebo>
-      <plugin name="${namespace}_${thruster_id}_thruster_model" filename="libuuv_thruster_ros_plugin.so">
+      <plugin name="uuv_simulator_ros::ThrusterROSPlugin" filename="libuuv_thruster_ros_plugin.so">
         <linkName>${namespace}/thruster_${thruster_id}</linkName>
         <jointName>${namespace}/thruster_${thruster_id}_joint</jointName>

Commit message: ROS2 migration updates and simulation changes

File: nps_uw_multibeam_sonar/urdf/multibeam_sonar_blueview_p900.xacro (robot description, xacro)
@@ -54,5 +54,5 @@
           </save> -->
         </camera>
-        <plugin filename="libnps_multibeam_sonar_ros_plugin.so" name="${name}_sensor_controller">
+        <plugin filename="libnps_multibeam_sonar_ros_plugin.so" name="nps_uw_multibeam_sonar::NpsGazeboRosMultibeamSonar">
           <!-- Sonar properties -->
           <verticalFOV>90</verticalFOV>
@@ -131,5 +131,5 @@
           </noise>
         </ray>
-        <plugin filename="libnps_multibeam_sonar_ray_ros_plugin.so" name="${name}_sensor_controller">
+        <plugin filename="libnps_multibeam_sonar_ray_ros_plugin.so" name="nps_uw_multibeam_sonar::NpsGazeboRosMultibeamSonarRay">
           <!-- Sonar properties -->
           <verticalFOV>90</verticalFOV>

File: rexrov2/rexrov2_description/urdf/rexrov2_base.xacro (robot description, xacro)
@@ -68,8 +68,8 @@
           <origin xyz="-4.8 0 0.05" rpy="0 1.57079632679 0"/>
           <geometry>
-            <cylinder radius="0.78" length="8.6"/>
+            <cylinder radius="0.08" length="8.6"/>
           </geometry>
           <material name="eroas_wake_green">
-            <color rgba="0.0 0.85 0.45 0.95"/>
+            <color rgba="0.0 1.0 0.3 0.3"/>
           </material>
         </visual>
@@ -77,8 +77,8 @@
           <origin xyz="-9.1 0 0.05" rpy="0 0 0"/>
           <geometry>
-            <sphere radius="0.78"/>
+            <sphere radius="0.08"/>
           </geometry>
           <material name="eroas_wake_green">
-            <color rgba="0.0 0.85 0.45 0.95"/>
+            <color rgba="0.0 1.0 0.3 0.3"/>
           </material>
         </visual>

File: uuv_simulator/uuv_gazebo_plugins/uuv_gazebo_ros_plugins/urdf/thruster_snippets.xacro (robot description, xacro)
@@ -102,5 +102,5 @@
     </link>
     <gazebo>
-      <plugin name="${namespace}_${thruster_id}_thruster_model" filename="libuuv_thruster_ros_plugin.so">
+      <plugin name="uuv_simulator_ros::ThrusterROSPlugin" filename="libuuv_thruster_ros_plugin.so">
         <linkName>${namespace}/thruster_${thruster_id}</linkName>
         <jointName>${namespace}/thruster_${thruster_id}_joint</jointName>
