Commit message: Fix ROS2 EROAS World A sonar and contour navigation

File: nps_uw_multibeam_sonar/urdf/multibeam_sonar_blueview_p900.xacro (robot description, xacro)
@@ -92,9 +92,13 @@
                gaussian_noise_mean gaussian_noise_stddev fidelity debug">
     <gazebo reference="${sensor_link}">
-      <sensor name="${name}_sensor" type="gpu_ray">
-        <visualize>false</visualize>
+      <!-- Gazebo Harmonic uses the GPU lidar sensor/component path.  Keep the
+           historical "ray" macro name for launch compatibility, but generate
+           Harmonic SDF so the NPS plugin can attach to GpuLidarSensor. -->
+      <sensor name="${name}_sensor" type="gpu_lidar">
+        <visualize>true</visualize>
         <always_on>true</always_on>
         <update_rate>10</update_rate>
-        <ray>
+        <lidar>
+          <visualize>true</visualize>
           <scan>
             <!-- Set horizontal FOV by setting image height -->
@@ -130,5 +134,5 @@
             <stddev>${gaussian_noise_stddev}</stddev>
           </noise>
-        </ray>
+        </lidar>
         <plugin filename="libnps_multibeam_sonar_ray_ros_plugin.so" name="nps_uw_multibeam_sonar::NpsGazeboRosMultibeamSonarRay">
           <!-- Sonar properties -->
@@ -139,4 +143,8 @@
           <sourceLevel>220</sourceLevel>
           <maxDistance>${maxDistance}</maxDistance>
+          <!-- Harmonic's GpuLidar can return the sonar housing / RexROV hull
+               while the vertical joint is pivoted.  Reject only that
+               near-field self-occlusion before synthesizing the sonar image. -->
+          <pointCloudCutoff>0.30</pointCloudCutoff>
           <raySkips>${raySkips}</raySkips>
           <sensorGain>${sensorGain}</sensorGain>
@@ -177,12 +185,15 @@
   <xacro:macro name="multibeam_blueview_p900_visual_ray" params="name ray_visual">
     <gazebo reference="${name}_visual_ray_link">
-      <sensor type="ray" name="multibeam_ray">
+      <sensor type="gpu_lidar" name="multibeam_ray">
         <pose>0 0 0 0 0 0</pose>
-        <update_rate>5</update_rate>
+        <update_rate>8</update_rate>
         <visualize>${ray_visual}</visualize>
-        <ray>
+        <always_on>true</always_on>
+        <topic>/rexrov2/sonar_visual_rays</topic>
+        <lidar>
+          <visualize>${ray_visual}</visualize>
           <scan>
             <horizontal>
-              <samples>100</samples>
+              <samples>120</samples>
               <resolution>1</resolution>
               <min_angle>-0.785398</min_angle>
@@ -201,5 +212,5 @@
             <resolution>0.01</resolution>
           </range>
-        </ray>
+        </lidar>
       </sensor>
     </gazebo>

File: rexrov2/rexrov2_description/urdf/rexrov2_sensors.xacro (robot description, xacro)
@@ -88,6 +88,28 @@
     <origin xyz="1.3 0 0.615" rpy="3.141592 0 0"/>
     <axis xyz="0 1 0"/> <!-- Rotation around Y-axis , check if this is correct-->
-    <limit effort="100" lower="-1.5708" upper="1.5708" velocity="100"/> <!-- 0 to 90 degrees in radians -->
+    <limit effort="100" lower="-1.5708" upper="1.5708" velocity="8.0"/>
+    <dynamics damping="0.8" friction="0.05"/>
   </joint>
+  <!-- Gazebo Harmonic replacement for the Gazebo Classic ROS joint
+       position controller.  ROS commands are bridged to this Gazebo topic
+       by start_EROAS_demo.launch.py. -->
+  <gazebo>
+    <plugin filename="gz-sim-joint-position-controller-system"
+            name="gz::sim::systems::JointPositionController">
+      <joint_name>${namespace}/sonar_vertical_joint</joint_name>
+      <topic>/${namespace}/sonar_joint_position_controller/command</topic>
+      <!-- The force-command PID is unstable for this lightweight sonar link
+           in gz-sim 8.  Drive the position error through a bounded velocity
+           command so every Algorithm-1 elevation sample can settle. -->
+      <use_velocity_commands>true</use_velocity_commands>
+      <p_gain>2.0</p_gain>
+      <i_gain>0.0</i_gain>
+      <d_gain>0.0</d_gain>
+      <i_max>0.0</i_max>
+      <i_min>0.0</i_min>
+      <cmd_max>0.8</cmd_max>
+      <cmd_min>-0.8</cmd_min>
+    </plugin>
+  </gazebo>
   <transmission name="${namespace}/sonar_vertical_transmission">
     <type>transmission_interface/SimpleTransmission</type>
