Commit message: Configure RexROV simulation and world launch setup

File: rexrov2/rexrov2_description/robots/rexrov2_default.xacro (robot description, xacro)
@@ -17,4 +17,6 @@
   <xacro:arg name="use_simplified_mesh" default="false"/>
   <xacro:arg name="inertial_reference_frame" default="world"/>
+  <xacro:arg name="hover_mode" default="false"/>
+  <xacro:arg name="green_wake" default="false"/>
   <!-- Include the ROV macro file -->
   <xacro:include filename="$(find rexrov2_description)/urdf/rexrov2_base.xacro"/>
@@ -24,5 +26,6 @@
     namespace="$(arg namespace)"
     use_simplified_mesh="$(arg use_simplified_mesh)"
-    inertial_reference_frame="$(arg inertial_reference_frame)">
+    inertial_reference_frame="$(arg inertial_reference_frame)"
+    green_wake="$(arg green_wake)">
     <!--
       The underwater object plugin is given as an input block parameter to
@@ -30,14 +33,36 @@
     -->
     <gazebo>
-      <plugin name="uuv_plugin" filename="libuuv_underwater_object_ros_plugin.so">
-        <fluid_density>1028.0</fluid_density>
-        <flow_velocity_topic>hydrodynamics/current_velocity</flow_velocity_topic>
-        <debug>$(arg debug)</debug>
-        <!-- Adding the hydrodynamic and hydrostatic parameters for the vehicle-->
-        <xacro:rexrov2_hydro_model namespace="$(arg namespace)"/>
-      </plugin>
+      <xacro:unless value="$(arg hover_mode)">
+        <plugin name="uuv_simulator_ros::UnderwaterObjectROSPlugin" filename="libuuv_underwater_object_ros_plugin.so">
+          <fluid_density>1028.0</fluid_density>
+          <flow_velocity_topic>hydrodynamics/current_velocity</flow_velocity_topic>
+          <debug>$(arg debug)</debug>
+          <!-- Adding the hydrodynamic and hydrostatic parameters for the vehicle-->
+          <xacro:rexrov2_hydro_model namespace="$(arg namespace)"/>
+        </plugin>
+      </xacro:unless>
     </gazebo>
   </xacro:rexrov2_base>
+  <xacro:if value="$(arg hover_mode)">
+    <gazebo reference="$(arg namespace)/base_link">
+      <gravity>false</gravity>
+    </gazebo>
+  </xacro:if>
   <!-- Joint state publisher plugin -->
   <xacro:default_joint_state_publisher namespace="$(arg namespace)" update_rate="50"/>
+  <!-- Gazebo Harmonic systems used by the ROS 2 EROAS demo path. -->
+  <gazebo>
+    <plugin filename="gz-sim-velocity-control-system"
+            name="gz::sim::systems::VelocityControl">
+      <topic>/rexrov2/cmd_vel</topic>
+      <initial_linear>0 0 0</initial_linear>
+      <initial_angular>0 0 0</initial_angular>
+    </plugin>
+    <plugin filename="gz-sim-odometry-publisher-system"
+            name="gz::sim::systems::OdometryPublisher">
+      <dimensions>3</dimensions>
+      <odom_publish_frequency>30</odom_publish_frequency>
+      <odom_topic>/rexrov2/pose_gt</odom_topic>
+    </plugin>
+  </gazebo>
 </robot>

File: rexrov2/rexrov2_description/urdf/rexrov2.gazebo.xacro (robot description, xacro)
@@ -23,5 +23,5 @@
     <xacro:macro name="rexrov2_hydro_model" params="namespace">
         <link name="${namespace}/base_link">
-            <neutrally_buoyant>0</neutrally_buoyant>
+            <neutrally_buoyant>1</neutrally_buoyant>
             <volume>${volume}</volume>
             <box>

File: rexrov2/rexrov2_description/urdf/rexrov2_base.xacro (robot description, xacro)
@@ -22,5 +22,5 @@
   <xacro:property name="mass" value="1862.87"/>
   <xacro:macro name="rexrov2_base"
-    params="namespace *gazebo use_simplified_mesh inertial_reference_frame">
+    params="namespace *gazebo use_simplified_mesh inertial_reference_frame green_wake:=false">
     <!-- Defining base link according to ROS conventions: x forward, z up -->
     <link name="${namespace}/base_link">
@@ -64,4 +64,24 @@
         </visual>
       </xacro:unless>
+      <xacro:if value="${green_wake}">
+        <visual name="eroas_green_wake">
+          <origin xyz="-4.8 0 0.05" rpy="0 1.57079632679 0"/>
+          <geometry>
+            <cylinder radius="0.78" length="8.6"/>
+          </geometry>
+          <material name="eroas_wake_green">
+            <color rgba="0.0 0.85 0.45 0.95"/>
+          </material>
+        </visual>
+        <visual name="eroas_green_wake_cap">
+          <origin xyz="-9.1 0 0.05" rpy="0 0 0"/>
+          <geometry>
+            <sphere radius="0.78"/>
+          </geometry>
+          <material name="eroas_wake_green">
+            <color rgba="0.0 0.85 0.45 0.95"/>
+          </material>
+        </visual>
+      </xacro:if>
       <!-- bottom plate -->
       <collision>

Commit message: ROS2 Harmonic migration updates

File: rexrov2/rexrov2_description/robots/rexrov2_default.xacro (robot description, xacro)
@@ -19,7 +19,13 @@
   <xacro:arg name="hover_mode" default="false"/>
   <xacro:arg name="green_wake" default="false"/>
+  <xacro:arg name="use_velocity_control_plugin" default="true"/>
   <!-- Include the ROV macro file -->
   <xacro:include filename="$(find rexrov2_description)/urdf/rexrov2_base.xacro"/>
   <xacro:include filename="$(find rexrov2_description)/urdf/rexrov2.gazebo.xacro"/>
+  <xacro:macro name="disable_link_gravity" params="link_name">
+    <gazebo reference="${link_name}">
+      <gravity>false</gravity>
+    </gazebo>
+  </xacro:macro>
   <!-- Create the rexrov2 -->
   <xacro:rexrov2_base
@@ -45,7 +51,32 @@
   </xacro:rexrov2_base>
   <xacro:if value="$(arg hover_mode)">
-    <gazebo reference="$(arg namespace)/base_link">
-      <gravity>false</gravity>
-    </gazebo>
+    <xacro:disable_link_gravity link_name="$(arg namespace)/base_link"/>
+    <xacro:disable_link_gravity link_name="$(arg namespace)/dvl_link"/>
+    <xacro:disable_link_gravity link_name="$(arg namespace)/dvl_sonar0_link"/>
+    <xacro:disable_link_gravity link_name="$(arg namespace)/dvl_sonar1_link"/>
+    <xacro:disable_link_gravity link_name="$(arg namespace)/dvl_sonar2_link"/>
+    <xacro:disable_link_gravity link_name="$(arg namespace)/dvl_sonar3_link"/>
+    <xacro:disable_link_gravity link_name="$(arg namespace)/magnetometer_link"/>
+    <xacro:disable_link_gravity link_name="$(arg namespace)/rpt_link"/>
+    <xacro:disable_link_gravity link_name="$(arg namespace)/pressure_link"/>
+    <xacro:disable_link_gravity link_name="$(arg namespace)/imu_link"/>
+    <xacro:disable_link_gravity link_name="$(arg namespace)/camera_link"/>
+    <xacro:disable_link_gravity link_name="$(arg namespace)/camera_link_optical"/>
+    <xacro:disable_link_gravity link_name="$(arg namespace)/cameraright_link"/>
+    <xacro:disable_link_gravity link_name="$(arg namespace)/cameraright_link_optical"/>
+    <xacro:disable_link_gravity link_name="$(arg namespace)/cameraleft_link"/>
+    <xacro:disable_link_gravity link_name="$(arg namespace)/cameraleft_link_optical"/>
+    <xacro:disable_link_gravity link_name="$(arg namespace)/gps_link"/>
+    <xacro:disable_link_gravity link_name="$(arg namespace)/pose_sensor_link_default"/>
+    <xacro:disable_link_gravity link_name="$(arg namespace)/cc_sensor_link"/>
+    <xacro:disable_link_gravity link_name="$(arg namespace)/sonar_link"/>
+    <xacro:disable_link_gravity link_name="blueview_p900_link"/>
+    <xacro:disable_link_gravity link_name="blueview_p900_visual_ray_link"/>
+    <xacro:disable_link_gravity link_name="$(arg namespace)/thruster_0"/>
+    <xacro:disable_link_gravity link_name="$(arg namespace)/thruster_1"/>
+    <xacro:disable_link_gravity link_name="$(arg namespace)/thruster_2"/>
+    <xacro:disable_link_gravity link_name="$(arg namespace)/thruster_3"/>
+    <xacro:disable_link_gravity link_name="$(arg namespace)/thruster_4"/>
+    <xacro:disable_link_gravity link_name="$(arg namespace)/thruster_5"/>
   </xacro:if>
   <!-- Joint state publisher plugin -->
@@ -53,15 +84,18 @@
   <!-- Gazebo Harmonic systems used by the ROS 2 EROAS demo path. -->
   <gazebo>
-    <plugin filename="gz-sim-velocity-control-system"
-            name="gz::sim::systems::VelocityControl">
-      <topic>/rexrov2/cmd_vel</topic>
-      <initial_linear>0 0 0</initial_linear>
-      <initial_angular>0 0 0</initial_angular>
-    </plugin>
+    <xacro:if value="$(arg use_velocity_control_plugin)">
+      <plugin filename="gz-sim-velocity-control-system"
+              name="gz::sim::systems::VelocityControl">
+        <topic>/rexrov2/cmd_vel</topic>
+        <initial_linear>0 0 0</initial_linear>
+        <initial_angular>0 0 0</initial_angular>
+      </plugin>
+    </xacro:if>
     <plugin filename="gz-sim-odometry-publisher-system"
             name="gz::sim::systems::OdometryPublisher">
       <dimensions>3</dimensions>
       <odom_publish_frequency>30</odom_publish_frequency>
-      <odom_topic>/rexrov2/pose_gt</odom_topic>
+      <odom_frame>$(arg namespace)/odom</odom_frame>
+      <robot_base_frame>$(arg namespace)/base_link</robot_base_frame>
     </plugin>
   </gazebo>
